Commit message: Uncomment + inertial

File: description/robot_core.xacro (robot description, xacro)
@@ -1,5 +1,5 @@
 <?xml version="1.0"?>
 <robot xmlns:xacro="http://www.ros.org/wiki/xacro" >
-    <!-- <xacro:include filename="inertial_macros.xacro"/> -->
+    <xacro:include filename="inertial_macros.xacro"/>
     <xacro:property name="chassis_length" value="0.335"/>
     <xacro:property name="chassis_width" value="0.265"/>
@@ -9,5 +9,5 @@
     <xacro:property name="wheel_thickness" value="0.026"/>
     <xacro:property name="wheel_mass" value="0.05"/>
-    <xacro:property name="wheel_offset_x" value="0.226"/>
+    <xacro:property name="back_wheel_offset_x" value="0.226"/>
     <xacro:property name="wheel_offset_y" value="0.1485"/>
     <xacro:property name="wheel_offset_z" value="0.01"/>
@@ -46,5 +46,5 @@
         <parent link="base_link"/>
         <child link="chassis"/>
-        <origin xyz="${-wheel_offset_x} 0 ${-wheel_offset_z}"/>
+        <origin xyz="${-back_wheel_offset_x} 0 ${-wheel_offset_z}"/>
     </joint>
     <link name="chassis">
@@ -62,7 +62,8 @@
             </geometry>
         </collision>
-        <!-- <xacro:inertial_box mass="0.5" x="${chassis_length}" y="${chassis_width}" z="${chassis_height}">
+        <xacro:inertial_box mass="0.5" x="${chassis_length}" y="${chassis_width}" z="${chassis_height}">
+            <!-- origin should match visual origin -->
             <origin xyz="${chassis_length/2} 0 ${chassis_height/2}" rpy="0 0 0"/>
-        </xacro:inertial_box> -->
+        </xacro:inertial_box>
     </link>
     <gazebo reference="chassis">
@@ -70,11 +71,11 @@
     </gazebo>
     <!-- BACK LEFT WHEEL LINK -->
-    <joint name="left_wheel_joint" type="continuous">
+    <joint name="back_left_wheel_joint" type="continuous">
         <parent link="base_link"/>
-        <child link="left_wheel"/>
+        <child link="back_left_wheel"/>
         <origin xyz="0 ${wheel_offset_y} 0" rpy="-${pi/2} 0 0" />
         <axis xyz="0 0 1"/>
     </joint>
-    <link name="left_wheel">
+    <link name="back_left_wheel">
         <visual>
             <geometry>
@@ -88,20 +89,21 @@
             </geometry>
         </collision>
-        <!-- <xacro:inertial_cylinder mass="${wheel_mass}" length="${wheel_thickness}" radius="${wheel_radius}">
+        <xacro:inertial_cylinder mass="${wheel_mass}" length="${wheel_thickness}" radius="${wheel_radius}">
+            <!-- origin should match visual origin -->
             <origin xyz="0 0 0" rpy="0 0 0"/>
-        </xacro:inertial_cylinder> -->
+        </xacro:inertial_cylinder>
     </link>
-    <gazebo reference="left_wheel">
+    <gazebo reference="back_left_wheel">
         <material>Gazebo/Blue</material>
     </gazebo>
     <!-- FRONT LEFT WHEEL LINK -->
     <!-- BACK RIGHT WHEEL LINK -->
-    <joint name="right_wheel_joint" type="continuous">
+    <joint name="back_right_wheel_joint" type="continuous">
         <parent link="base_link"/>
-        <child link="right_wheel"/>
+        <child link="back_right_wheel"/>
         <origin xyz="0 ${-wheel_offset_y} 0" rpy="${pi/2} 0 0" />
         <axis xyz="0 0 -1"/>
     </joint>
-    <link name="right_wheel">
+    <link name="back_right_wheel">
         <visual>
             <geometry>
@@ -115,9 +117,10 @@
             </geometry>
         </collision>
-        <!-- <xacro:inertial_cylinder mass="${wheel_mass}" length="${wheel_thickness}" radius="${wheel_radius}">
+        <xacro:inertial_cylinder mass="${wheel_mass}" length="${wheel_thickness}" radius="${wheel_radius}">
+            <!-- origin should match visual origin -->
             <origin xyz="0 0 0" rpy="0 0 0"/>
-        </xacro:inertial_cylinder> -->
+        </xacro:inertial_cylinder>
     </link>
-    <gazebo reference="right_wheel">
+    <gazebo reference="back_right_wheel">
         <material>Gazebo/Blue</material>
     </gazebo>
@@ -141,7 +144,8 @@
             </geometry>
         </collision>
-        <!-- <xacro:inertial_sphere mass="${caster_wheel_mass}" radius="${caster_wheel_radius}">
+        <xacro:inertial_sphere mass="${caster_wheel_mass}" radius="${caster_wheel_radius}">
+            <!-- origin should match visual origin -->
             <origin xyz="0 0 0" rpy="0 0 0"/>
-        </xacro:inertial_sphere> -->
+        </xacro:inertial_sphere>
     </link>
     <gazebo reference="caster_wheel">

Commit message: updates

File: description/robot_core.xacro (robot description, xacro)
@@ -1,4 +1,5 @@
 <?xml version="1.0"?>
 <robot xmlns:xacro="http://www.ros.org/wiki/xacro" >
+    <!-- UNITS: Metric units for everything. Kilograms for mass and Meters for length -->
     <xacro:include filename="inertial_macros.xacro"/>
     <xacro:property name="chassis_length" value="0.335"/>
@@ -12,5 +13,5 @@
     <xacro:property name="wheel_offset_y" value="0.1485"/>
     <xacro:property name="wheel_offset_z" value="0.01"/>
-    <xacro:property name="caster_wheel_radius" value="0.01"/>
+    <xacro:property name="caster_wheel_radius" value="0.05"/>
     <xacro:property name="caster_wheel_mass" value="0.01"/>
     <xacro:property name="caster_wheel_offset_x" value="0.075"/>

Commit message: Front Right Wheel Proto

File: description/robot_core.xacro (robot description, xacro)
@@ -10,4 +10,5 @@
     <xacro:property name="wheel_thickness" value="0.026"/>
     <xacro:property name="wheel_mass" value="0.05"/>
+    <xacro:property name="front_wheel_offset_x" value="0.25"/>
     <xacro:property name="back_wheel_offset_x" value="0.226"/>
     <xacro:property name="wheel_offset_y" value="0.1485"/>
@@ -127,4 +128,30 @@
     </gazebo>
     <!-- FRONT RIGHT WHEEL LINK -->
+    <joint name="front_right_wheel_joint" type="continuous">
+        <parent link="base_link"/>
+        <child link="front_right_wheel"/>
+        <origin xyz="${front_wheel_offset_x} ${-wheel_offset_y} 0" rpy="${pi/2} 0 0" />
+        <axis xyz="0 0 -1"/>
+    </joint>
+    <link name="front_right_wheel">
+        <visual>
+            <geometry>
+                <cylinder radius="${wheel_radius}" length="${wheel_thickness}"/>
+            </geometry>
+            <material name="blue"/>
+        </visual>
+        <collision>
+            <geometry>
+                <sphere radius="${wheel_radius}"/>
+            </geometry>
+        </collision>
+        <xacro:inertial_cylinder mass="${wheel_mass}" length="${wheel_thickness}" radius="${wheel_radius}">
+            <!-- origin should match visual origin -->
+            <origin xyz="0 0 0" rpy="0 0 0"/>
+        </xacro:inertial_cylinder>
+    </link>
+    <gazebo reference="front_right_wheel">
+        <material>Gazebo/Blue</material>
+    </gazebo>
     <!-- CASTER WHEEL LINK -->
     <joint name="caster_wheel_joint" type="fixed">

Commit message: Front Wheels Added to Model

File: description/robot_core.xacro (robot description, xacro)
@@ -10,6 +10,6 @@
     <xacro:property name="wheel_thickness" value="0.026"/>
     <xacro:property name="wheel_mass" value="0.05"/>
-    <xacro:property name="front_wheel_offset_x" value="0.25"/>
-    <xacro:property name="back_wheel_offset_x" value="0.226"/>
+    <xacro:property name="front_wheel_offset_x" value="0.2"/>
+    <xacro:property name="back_wheel_offset_x" value="0.3"/>
     <xacro:property name="wheel_offset_y" value="0.1485"/>
     <xacro:property name="wheel_offset_z" value="0.01"/>
@@ -100,4 +100,30 @@
     </gazebo>
     <!-- FRONT LEFT WHEEL LINK -->
+    <joint name="front_left_wheel_joint" type="continuous">
+        <parent link="base_link"/>
+        <child link="front_left_wheel"/>
+        <origin xyz="${-front_wheel_offset_x} ${wheel_offset_y} 0" rpy="-${pi/2} 0 0" />
+        <axis xyz="0 0 1"/>
+    </joint>
+    <link name="front_left_wheel">
+        <visual>
+            <geometry>
+                <cylinder radius="${wheel_radius}" length="${wheel_thickness}"/>
+            </geometry>
+            <material name="blue"/>
+        </visual>
+        <collision>
+            <geometry>
+                <sphere radius="${wheel_radius}"/>
+            </geometry>
+        </collision>
+        <xacro:inertial_cylinder mass="${wheel_mass}" length="${wheel_thickness}" radius="${wheel_radius}">
+            <!-- origin should match visual origin -->
+            <origin xyz="0 0 0" rpy="0 0 0"/>
+        </xacro:inertial_cylinder>
+    </link>
+    <gazebo reference="front_left_wheel">
+        <material>Gazebo/Blue</material>
+    </gazebo>
     <!-- BACK RIGHT WHEEL LINK -->
     <joint name="back_right_wheel_joint" type="continuous">
@@ -131,5 +157,5 @@
         <parent link="base_link"/>
         <child link="front_right_wheel"/>
-        <origin xyz="${front_wheel_offset_x} ${-wheel_offset_y} 0" rpy="${pi/2} 0 0" />
+        <origin xyz="${-front_wheel_offset_x} ${-wheel_offset_y} 0" rpy="${pi/2} 0 0" />
         <axis xyz="0 0 -1"/>
     </joint>
@@ -154,31 +180,3 @@
         <material>Gazebo/Blue</material>
     </gazebo>
-    <!-- CASTER WHEEL LINK -->
-    <joint name="caster_wheel_joint" type="fixed">
-        <parent link="chassis"/>
-        <child link="caster_wheel"/>
-        <origin xyz="${caster_wheel_offset_x} 0 ${caster_wheel_offset_z}"/>
-    </joint>
-    <link name="caster_wheel">
-        <visual>
-            <geometry>
-                <sphere radius="${caster_wheel_radius}"/>
-            </geometry>
-            <material name="white"/>
-        </visual>
-        <collision>
-            <geometry>
-                <sphere radius="${caster_wheel_radius}"/>
-            </geometry>
-        </collision>
-        <xacro:inertial_sphere mass="${caster_wheel_mass}" radius="${caster_wheel_radius}">
-            <!-- origin should match visual origin -->
-            <origin xyz="0 0 0" rpy="0 0 0"/>
-        </xacro:inertial_sphere>
-    </link>
-    <gazebo reference="caster_wheel">
-        <material>Gazebo/White</material>
-        <mu1 value="0.001"/>
-        <mu2 value="0.001"/>
-    </gazebo>
 </robot>

Commit message: Measurements modified

File: description/robot_core.xacro (robot description, xacro)
@@ -3,19 +3,15 @@
     <!-- UNITS: Metric units for everything. Kilograms for mass and Meters for length -->
     <xacro:include filename="inertial_macros.xacro"/>
-    <xacro:property name="chassis_length" value="0.335"/>
-    <xacro:property name="chassis_width" value="0.265"/>
-    <xacro:property name="chassis_height" value="0.138"/>
+    <xacro:property name="chassis_length" value="0.3556"/>
+    <xacro:property name="chassis_width" value="0.2032"/>
+    <xacro:property name="chassis_height" value="0.3556"/>
     <xacro:property name="chassis_mass" value="1.0"/>
-    <xacro:property name="wheel_radius" value="0.033"/>
-    <xacro:property name="wheel_thickness" value="0.026"/>
+    <xacro:property name="wheel_radius" value="0.0762"/>
+    <xacro:property name="wheel_thickness" value="0.0254"/>
     <xacro:property name="wheel_mass" value="0.05"/>
-    <xacro:property name="front_wheel_offset_x" value="0.2"/>
-    <xacro:property name="back_wheel_offset_x" value="0.3"/>
-    <xacro:property name="wheel_offset_y" value="0.1485"/>
-    <xacro:property name="wheel_offset_z" value="0.01"/>
-    <xacro:property name="caster_wheel_radius" value="0.05"/>
-    <xacro:property name="caster_wheel_mass" value="0.01"/>
-    <xacro:property name="caster_wheel_offset_x" value="0.075"/>
-    <xacro:property name="caster_wheel_offset_z" value="${wheel_offset_z - wheel_radius + caster_wheel_radius}"/>
+    <xacro:property name="front_wheel_offset_x" value="0.291465"/>
+    <xacro:property name="back_wheel_offset_x" value="0.064135"/>
+    <xacro:property name="wheel_offset_y" value="0.1143"/>
+    <xacro:property name="wheel_offset_z" value="0.026035"/>
     <material name="white">
         <color rgba="1 1 1 1" />

Commit message: More 3D modeling work

File: description/robot_core.xacro (robot description, xacro)
@@ -10,6 +10,6 @@
     <xacro:property name="wheel_thickness" value="0.0254"/>
     <xacro:property name="wheel_mass" value="0.05"/>
-    <xacro:property name="front_wheel_offset_x" value="0.291465"/>
-    <xacro:property name="back_wheel_offset_x" value="0.064135"/>
+    <xacro:property name="front_wheel_offset_x" value="0.22733"/>
+    <xacro:property name="back_wheel_offset_x" value="0.291465"/>
     <xacro:property name="wheel_offset_y" value="0.1143"/>
     <xacro:property name="wheel_offset_z" value="0.026035"/>
@@ -24,8 +24,14 @@
     </material>
     <material name="black">
-        <color rgba="0 0 0 1"/>
+        <color rgba="0.25 0.25 0.25 1"/>
     </material>
     <material name="red">
         <color rgba="1 0 0 1"/>
+    </material>
+    <material name="gray">
+        <color rgba="0.8 0.8 0.8 1"/>
+    </material>
+    <material name="gold">
+        <color rgba="1 0.84 0 1"/>
     </material>
     <!-- BASE LINK -->
@@ -52,5 +58,5 @@
                 <box size="${chassis_length} ${chassis_width} ${chassis_height}"/>
             </geometry>
-            <material name="orange"/>
+            <material name="black"/>
         </visual>
         <collision>
@@ -66,5 +72,5 @@
     </link>
     <gazebo reference="chassis">
-        <material>Gazebo/Orange</material>
+        <material>Gazebo/Black</material>
     </gazebo>
     <!-- BACK LEFT WHEEL LINK -->
@@ -80,5 +86,5 @@
                 <cylinder radius="${wheel_radius}" length="${wheel_thickness}"/>
             </geometry>
-            <material name="blue"/>
+            <material name="gray"/>
         </visual>
         <collision>
@@ -93,5 +99,5 @@
     </link>
     <gazebo reference="back_left_wheel">
-        <material>Gazebo/Blue</material>
+        <material>Gazebo/Gray</material>
     </gazebo>
     <!-- FRONT LEFT WHEEL LINK -->
@@ -107,5 +113,5 @@
                 <cylinder radius="${wheel_radius}" length="${wheel_thickness}"/>
             </geometry>
-            <material name="blue"/>
+            <material name="gray"/>
         </visual>
         <collision>
@@ -120,5 +126,5 @@
     </link>
     <gazebo reference="front_left_wheel">
-        <material>Gazebo/Blue</material>
+        <material>Gazebo/Gray</material>
     </gazebo>
     <!-- BACK RIGHT WHEEL LINK -->
@@ -134,5 +140,5 @@
                 <cylinder radius="${wheel_radius}" length="${wheel_thickness}"/>
             </geometry>
-            <material name="blue"/>
+            <material name="gray"/>
         </visual>
         <collision>
@@ -147,5 +153,5 @@
     </link>
     <gazebo reference="back_right_wheel">
-        <material>Gazebo/Blue</material>
+        <material>Gazebo/Gray</material>
     </gazebo>
     <!-- FRONT RIGHT WHEEL LINK -->
@@ -161,5 +167,5 @@
                 <cylinder radius="${wheel_radius}" length="${wheel_thickness}"/>
             </geometry>
-            <material name="blue"/>
+            <material name="gray"/>
         </visual>
         <collision>
@@ -174,5 +180,5 @@
     </link>
     <gazebo reference="front_right_wheel">
-        <material>Gazebo/Blue</material>
+        <material>Gazebo/Gray</material>
     </gazebo>
 </robot>

Commit message: chassis top

File: description/robot_core.xacro (robot description, xacro)
@@ -3,8 +3,12 @@
     <!-- UNITS: Metric units for everything. Kilograms for mass and Meters for length -->
     <xacro:include filename="inertial_macros.xacro"/>
-    <xacro:property name="chassis_length" value="0.3556"/>
-    <xacro:property name="chassis_width" value="0.2032"/>
-    <xacro:property name="chassis_height" value="0.3556"/>
-    <xacro:property name="chassis_mass" value="1.0"/>
+    <xacro:property name="chassis_base_length" value="0.3556"/>
+    <xacro:property name="chassis_base_width" value="0.2032"/>
+    <xacro:property name="chassis_base_height" value="0.1397"/>
+    <xacro:property name="chassis_base_mass" value="1.0"/>
+    <xacro:property name="chassis_top_length" value="0.4064"/>
+    <xacro:property name="chassis_top_width" value="0.254"/>
+    <xacro:property name="chassis_top_height" value="0.1905"/>
+    <xacro:property name="chassis_top_mass" value="1.0"/>
     <xacro:property name="wheel_radius" value="0.0762"/>
     <xacro:property name="wheel_thickness" value="0.0254"/>
@@ -46,32 +50,53 @@
     <link name="base_footprint">
     </link>
-    <!-- CHASSIS LINK -->
-    <joint name="chassis_joint" type="fixed">
-        <parent link="base_link"/>
-        <child link="chassis"/>
+    <!-- CHASSIS BASE LINK -->
+    <joint name="chassis_base_joint" type="fixed">
+        <parent link="base_link"/>
+        <child link="chassis_base"/>
         <origin xyz="${-back_wheel_offset_x} 0 ${-wheel_offset_z}"/>
     </joint>
-    <link name="chassis">
-        <visual>
-            <origin xyz="${chassis_length/2} 0 ${chassis_height/2}"/>
-            <geometry>
-                <box size="${chassis_length} ${chassis_width} ${chassis_height}"/>
+    <link name="chassis_base">
+        <visual>
+            <origin xyz="${chassis_base_length/2} 0 ${chassis_base_height/2}"/>
+            <geometry>
+                <box size="${chassis_base_length} ${chassis_base_width} ${chassis_base_height}"/>
             </geometry>
             <material name="black"/>
         </visual>
         <collision>
-            <origin xyz="${chassis_length/2} 0 ${chassis_height/2}"/>
-            <geometry>
-                <box size="${chassis_length} ${chassis_width} ${chassis_height}"/>
-            </geometry>
-        </collision>
-        <xacro:inertial_box mass="0.5" x="${chassis_length}" y="${chassis_width}" z="${chassis_height}">
-            <!-- origin should match visual origin -->
-            <origin xyz="${chassis_length/2} 0 ${chassis_height/2}" rpy="0 0 0"/>
+            <origin xyz="${chassis_base_length/2} 0 ${chassis_base_height/2}"/>
+            <geometry>
+                <box size="${chassis_base_length} ${chassis_base_width} ${chassis_base_height}"/>
+            </geometry>
+        </collision>
+        <xacro:inertial_box mass="0.5" x="${chassis_base_length}" y="${chassis_base_width}" z="${chassis_base_height}">
+            <!-- origin should match visual origin -->
+            <origin xyz="${chassis_base_length/2} 0 ${chassis_base_height/2}" rpy="0 0 0"/>
         </xacro:inertial_box>
     </link>
-    <gazebo reference="chassis">
+    <gazebo reference="chassis_base">
         <material>Gazebo/Black</material>
     </gazebo>
+    <!-- CHASSIS TOP LINK -->
+    <joint name="chassis_top_joint" type="fixed">
+        <origin xyz="0 0 0.1905" rpy="0 0 0" />
+        <parent link="chassis_base"/>
+        <child link="chassis_top"/>
+    </joint>
+    <link name="chassis_top">
+        <visual>
+            <origin xyz="0 0 0" rpy="0 0 0" />
+            <geometry>
+                <box size="${chassis_top_length} ${chassis_top_width} ${chassis_top_height}" />
+            </geometry>
+            <material name="gold" />
+        </visual>
+        <collision>
+            <origin xyz="0 0 0" rpy="0 0 0" />
+            <geometry>
+                <box size="${chassis_top_length} ${chassis_top_width} ${chassis_top_height}" />
+            </geometry>
+        </collision>
+    </link>
     <!-- BACK LEFT WHEEL LINK -->
     <joint name="back_left_wheel_joint" type="continuous">

Commit message: Chassis Top Correction

File: description/robot_core.xacro (robot description, xacro)
@@ -54,4 +54,5 @@
         <parent link="base_link"/>
         <child link="chassis_base"/>
+        <!-- change this so that the origin is on the complete back wall -->
         <origin xyz="${-back_wheel_offset_x} 0 ${-wheel_offset_z}"/>
     </joint>
@@ -80,5 +81,5 @@
     <!-- CHASSIS TOP LINK -->
     <joint name="chassis_top_joint" type="fixed">
-        <origin xyz="0 0 0.1905" rpy="0 0 0" />
+        <origin xyz="${chassis_base_length/2} 0 ${chassis_base_height}" rpy="0 0 0" />
         <parent link="chassis_base"/>
         <child link="chassis_top"/>
@@ -86,5 +87,5 @@
     <link name="chassis_top">
         <visual>
-            <origin xyz="0 0 0" rpy="0 0 0" />
+            <origin xyz="0 0 ${chassis_top_height/2}"/>
             <geometry>
                 <box size="${chassis_top_length} ${chassis_top_width} ${chassis_top_height}" />

Commit message: lid

File: description/robot_core.xacro (robot description, xacro)
@@ -100,4 +100,25 @@
         </collision>
     </link>
+    <!-- LID LINK -->
+    <joint name="lid_joint" type="fixed">
+        <origin xyz="0 0 ${chassis_top_height}" />
+        <parent link="chassis_top"/>
+        <child link="lid"/>
+    </joint>
+    <link name="lid">
+        <visual>
+            <origin xyz="0 0 ${chassis_top_height}" />
+            <geometry>
+                <box size="${chassis_top_length} ${chassis_top_width} ${chassis_top_height}" />
+            </geometry>
+            <material name="white" />
+        </visual>
+        <collision>
+            <origin xyz="0 0 ${chassis_top_height}" />
+            <geometry>
+                <box size="${chassis_top_length} ${chassis_top_width} ${chassis_top_height}" />
+            </geometry>
+        </collision>
+    </link>
     <!-- BACK LEFT WHEEL LINK -->
     <joint name="back_left_wheel_joint" type="continuous">

Commit message: Finalized URDF per video progress

File: description/robot_core.xacro (robot description, xacro)
@@ -11,4 +11,5 @@
     <xacro:property name="chassis_top_height" value="0.1905"/>
     <xacro:property name="chassis_top_mass" value="1.0"/>
+    <xacro:property name="lid_thickness" value="0.0254"/>
     <xacro:property name="wheel_radius" value="0.0762"/>
     <xacro:property name="wheel_thickness" value="0.0254"/>
@@ -100,4 +101,7 @@
         </collision>
     </link>
+    <gazebo reference="chassis_top">
+        <material>Gazebo/Black</material>
+    </gazebo>
     <!-- LID LINK -->
     <joint name="lid_joint" type="fixed">
@@ -108,17 +112,20 @@
     <link name="lid">
         <visual>
-            <origin xyz="0 0 ${chassis_top_height}" />
-            <geometry>
-                <box size="${chassis_top_length} ${chassis_top_width} ${chassis_top_height}" />
-            </geometry>
-            <material name="white" />
-        </visual>
-        <collision>
-            <origin xyz="0 0 ${chassis_top_height}" />
-            <geometry>
-                <box size="${chassis_top_length} ${chassis_top_width} ${chassis_top_height}" />
-            </geometry>
-        </collision>
-    </link>
+            <origin xyz="0 0 ${lid_thickness/2}" />
+            <geometry>
+                <box size="${chassis_top_length} ${chassis_top_width} ${lid_thickness}" />
+            </geometry>
+            <material name="black" />
+        </visual>
+        <collision>
+            <origin xyz="0 0 ${lid_thickness}" />
+            <geometry>
+                <box size="${chassis_top_length} ${chassis_top_width} ${lid_thickness}" />
+            </geometry>
+        </collision>
+    </link>
+    <gazebo reference="lid">
+        <material>Gazebo/Gold</material>
+    </gazebo>
     <!-- BACK LEFT WHEEL LINK -->
     <joint name="back_left_wheel_joint" type="continuous">
